Commit message: 新增 camera

File: ur_mir_data/mir_ur.urdf (robot description, URDF)
Before this commit: robot mir_100, 31 links, 30 joints
Links:
- added link view_link
Joints:
- added joint glass_to_view: type fixed, parent glass_link, child view_link, origin xyz=0.0 0.0 0.0 rpy=4.71225 4.71225 1.57075, axis 0.0 0.0 0.0
- joint base_to_camera: origin xyz=0.0 -0.05 -0.06 rpy=0.0 0.0 1.57075 -> xyz=0 0.03 0.06 rpy=0 3.1415 4.71225; parent base -> ur10_wrist_3_link

Commit message: 新增 Laser 和 map

File: ur_mir_data/mir_ur.urdf (robot description, URDF)
Before this commit: robot mir_100, 32 links, 31 joints
Links:
- link back_laser_link: geometry visual mesh filename=package://meshes/mir/visual/sick_lms-100.stl
- link front_laser_link: geometry visual mesh filename=package://meshes/mir/visual/sick_lms-100.stl
